File: KiCad Sources/1002_EPROM_EMU_NG/1002_EPROM_EMU_NG.sch (KiCad schematic (older format))
At the start: 40 parts, among them J1 IDC34, M1 Arduino Nano v3.0, Q1 BC547, Q2 BC557, SW1 SW_Push, U1 74HC00, U10 74HC541, U11 74HC541, U2 74HC08, U3 25LC512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

Commit message: Add files via upload
Parts:
- added TP1: VCC, TestPoint:TestPoint_THTPad_D1.5mm_Drill0.7mm, symbol Connector:TestPoint
- added TP2, TP3: GND, TestPoint:TestPoint_THTPad_D1.5mm_Drill0.7mm, symbol Connector:TestPoint
- C1: value 10uF -> 100uF
- F1: value Polyfuse_50mA -> Polyfuse_200mA
Connections:
- net GND: now also TP2.1, TP3.1
- net VCC: now also TP1.1
Other:
- note removed: "Q. But why are you using IDC34 for J1?\nA1. IDC34 was used in other popular kit so it's much cheaper vs IDC30\nA2. I had a commercial EMULATOR and wanted to re-use the "probe"."
- note removed: "Q. Why SPI EEPROM, you could have used Flash-based main memory instead of SRAM.\n\nA1. This was added last moment, had few spare pins, and thought might be useful to save state.\nA2. Have a commercial emulator based on SRAM and it works fine for the majority of my use cases.\nA3. SPI driver library is built into Arduino and I'm too lazy to write the Flash implementation?? :)\nA4. The SPI section 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"
- note removed: "Some RESET circuits are tricky to trigger with just a transistor, \nin that case, use a small relay and drive it with this transistor \n(don't forget about extra protection diode if it's not built into the relay already)."
- note removed: "You can skip the diode and polyfuse but:\n- 5V will flow to your device (remember current limit on Aruduino Nano)\n- You will not be protected from accidently reversing power polarity.\n\nYou will gain:\n- much less voltage drop if you want to power the emulator from target."
- moved on the sheet: C1, C2, C3, C4, C5, C6, C7, D3, D5, F1, H1, H2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

Commit message: Updated PCB to version 1.6
Parts:
- added H5: MountingHole, Symbol:OSHW-Logo2_9.8x8mm_SilkScreen, symbol Mechanical:MountingHole
- added TP4: VCC, TestPoint:TestPoint_THTPad_D1.5mm_Drill0.7mm, symbol Connector:TestPoint
- C1: value 100uF -> 10uF
- Q1: value BC547 -> 2N4401
- Q2: value BC557 -> 2N4403
- R4: value 10k -> 4k7
- U10, U11, U9: value 74HC541 -> 74HCT541
Connections:
- net E_RESET: now also J1.1 (Pin_1)
- net VCC: now also TP4.1
- net ~E_RESET~: now also J1.2 (Pin_2)
- no-connect marks 16 -> 14
Changed lines of the file:
@@
 	13700 4650 13700 4750
 Wire Wire Line
-	14950 3250 14600 3250
+	15000 3250 14650 3250
 $Comp
 L power:GND #PWR015
@@
 P 12400 2300
 F 0 "U9" H 12150 3050 50  0000 C CNN
-F 1 "74HC541" H 12250 2950 50  0000 C CNN
+F 1 "74HCT541" H 12250 2950 50  0000 C CNN
 F 2 "Package_DIP:DIP-20_W7.62mm_Socket" H 12400 2300 50  0001 C CNN
 F 3 "http://www.ti.com/lit/gpn/sn74LS541" H 12400 2300 50  0001 C CNN
@@
 P 12400 4150
 F 0 "U10" H 12150 4900 50  0000 C CNN
-F 1 "74HC541" H 12250 4800 50  0000 C CNN
+F 1 "74HCT541" H 12250 4800 50  0000 C CNN
 F 2 "Package_DIP:DIP-20_W7.62mm_Socket" H 12400 4150 50  0001 C CNN
 F 3 "http://www.ti.com/lit/gpn/sn74LS541" H 12400 4150 50  0001 C CNN
@@
 P 12400 5800
 F 0 "U11" H 12150 6550 50  0000 C CNN
-F 1 "74HC541" H 12250 6450 50  0000 C CNN
+F 1 "74HCT541" H 12250 6450 50  0000 C CNN
 F 2 "Package_DIP:DIP-20_W7.62mm_Socket" H 12400 5800 50  0001 C CNN
 F 3 "http://www.ti.com/lit/gpn/sn74LS541" H 12400 5800 50  0001 C CNN
@@
 Text Label 12950 2800 0    50   ~ 0
 E_~CS~
-Text Label 14950 3250 2    50   ~ 0
+Text Label 15000 3250 2    50   ~ 0
 E_RESET
-Text Label 13800 3250 0    50   ~ 0
+Text Label 13700 3250 0    50   ~ 0
 ~E_RESET~
 Wire Wire Line
-	13800 3250 14100 3250
+	13700 3250 14050 3250
 Entry Wire Line
 	13300 4450 13400 4550
@@
 	2800 4700 2450 4700
 $Comp
-L Device:C C2
-U 1 1 5FD67446
-P 4100 9300
-F 0 "C2" H 4150 9500 50  0000 L CNN
-F 1 "100nF" H 3850 9400 50  0001 L CNN
-F 2 "Capacitor_THT:C_Disc_D4.7mm_W2.5mm_P5.00mm" H 4138 9150 50  0001 C CNN
-F 3 "~" H 4100 9300 50  0001 C CNN
-	1    4100 9300
-	1    0    0    -1
-$EndComp
-$Comp
 L Device:CP_Small C1
 U 1 1 5FD68EF5
 P 2250 9250
 F 0 "C1" H 2000 9550 50  0000 L CNN
-F 1 "100uF" H 2000 9450 50  0000 L CNN
+F 1 "10uF" H 2000 9450 50  0000 L CNN
 F 2 "Capacitor_THT:CP_Radial_D6.3mm_P2.50mm" H 2250 9250 50  0001 C CNN
 F 3 "~" H 2250 9250 50  0001 C CNN
@@
 F 3 "~" H 5100 9300 50  0001 C CNN
 	1    5100 9300
-	1    0    0    -1
-$EndComp
-$Comp
-L Device:C C7
-U 1 1 5FFDC459
-P 5600 9300
-F 0 "C7" H 5650 9500 50  0000 L CNN
-F 1 "22nF" H 5650 9400 50  0000 L CNN
-F 2 "Capacitor_THT:C_Disc_D4.7mm_W2.5mm_P5.00mm" H 5638 9150 50  0001 C CNN
-F 3 "~" H 5600 9300 50  0001 C CNN
-	1    5600 9300
 	1    0    0    -1
 $EndComp
@@
 P 14200 8200
 F 0 "Q1" H 14391 8246 50  0000 L CNN
-F 1 "BC547" H 14391 8155 50  0000 L CNN
+F 1 "2N4401" H 14391 8155 50  0000 L CNN
 F 2 "Package_TO_SOT_THT:TO-92_Inline_Wide" H 14400 8300 50  0001 C CNN
 F 3 "~" H 14200 8200 50  0001 C CNN
@@
 P 14200 6850
 F 0 "Q2" H 14391 6804 50  0000 L CNN
-F 1 "BC557" H 14391 6895 50  0000 L CNN
+F 1 "2N4403" H 14391 6895 50  0000 L CNN
 F 2 "Package_TO_SOT_THT:TO-92_Inline_Wide" H 14400 6950 50  0001 C CNN
 F 3 "~" H 14200 6850 50  0001 C CNN
@@
 P 13800 8200
 F 0 "R4" V 13700 8100 50  0000 L CNN
-F 1 "10k" V 13900 8100 50  0000 L CNN
+F 1 "4k7" V 13900 8100 50  0000 L CNN
 F 2 "Resistor_THT:R_Axial_DIN0204_L3.6mm_D1.6mm_P7.62mm_Horizontal" V 13730 8200 50  0001 C CNN
 F 3 "~" H 13800 8200 50  0001 C CNN
@@
 	0    -1   1    0
 $EndComp
-NoConn ~ 14600 3050
-NoConn ~ 14100 3050
 Text Label 15100 7750 2    50   ~ 0
 ~E_RESET~
@@
 Connection ~ 2500 8800
 Wire Wire Line
-	2500 8800 2850 8800
+	2500 8800 2600 8800
 $Comp
 L Connector:TestPoint TP3
@@
 Text Label 4200 3800 2    50   ~ 0
 EN_RST
+Wire Wire Line
+	4300 2700 5400 2700
+Text Label 4150 4400 2    50   ~ 0
+~WE~
+$Comp
+L Connector:TestPoint TP4
+U 1 1 5F3BA202
+P 2600 8800
+F 0 "TP4" H 2700 8950 50  0001 L CNN
+F 1 "VCC" H 2700 8850 50  0001 L CNN
+F 2 "TestPoint:TestPoint_THTPad_D1.5mm_Drill0.7mm" H 2800 8800 50  0001 C CNN
+F 3 "~" H 2800 8800 50  0001 C CNN
+	1    2600 8800
+	1    0    0    -1
+$EndComp
+Connection ~ 2600 8800
+Wire Wire Line
+	2600 8800 2850 8800
+$Comp
+L Device:C C7
+U 1 1 5FFDC459
+P 5600 9300
+F 0 "C7" H 5650 9500 50  0000 L CNN
+F 1 "22nF" H 5650 9400 50  0000 L CNN
+F 2 "Capacitor_THT:C_Disc_D4.7mm_W2.5mm_P5.00mm" H 5638 9150 50  0001 C CNN
+F 3 "~" H 5600 9300 50  0001 C CNN
+	1    5600 9300
+	1    0    0    -1
+$EndComp
+$Comp
+L Device:C C2
+U 1 1 5FD67446
+P 4100 9300
+F 0 "C2" H 4150 9500 50  0000 L CNN
+F 1 "100nF" H 3850 9400 50  0001 L CNN
+F 2 "Capacitor_THT:C_Disc_D4.7mm_W2.5mm_P5.00mm" H 4138 9150 50  0001 C CNN
+F 3 "~" H 4100 9300 50  0001 C CNN
+	1    4100 9300
+	1    0    0    -1
+$EndComp
+Wire Wire Line
+	14650 3250 14650 3050
+Wire Wire Line
+	14650 3050 14600 3050
+Connection ~ 14650 3250
+Wire Wire Line
+	14650 3250 14600 3250
+Wire Wire Line
+	14050 3250 14050 3050
+Wire Wire Line
+	14050 3050 14100 3050
+Connection ~ 14050 3250
+Wire Wire Line
+	14050 3250 14100 3250
+$Comp
+L Mechanical:MountingHole H5
+U 1 1 5F96F8A9
+P 9600 9550
+F 0 "H5" H 9700 9596 50  0001 L CNN
+F 1 "MountingHole" H 9700 9505 50  0001 L CNN
+F 2 "Symbol:OSHW-Logo2_9.8x8mm_SilkScreen" H 9600 9550 50  0001 C CNN
+F 3 "~" H 9600 9550 50  0001 C CNN
+	1    9600 9550
+	1    0    0    -1
+$EndComp
 Wire Bus Line
 	9400 2850 9400 4700
@@
 	8850 5400 8850 7750
 Wire Bus Line
+	9050 2300 9050 3900
+Wire Bus Line
+	15150 1200 15150 4550
+Wire Bus Line
 	7200 900  7200 2300
-Wire Bus Line
-	9050 2300 9050 3900
 Wire Bus Line
 	11400 900  11400 3900
 Wire Bus Line
 	13300 1200 13300 5900
-Wire Bus Line
-	15150 1200 15150 4550
-Wire Wire Line
-	4300 2700 5400 2700
-Text Label 4150 4400 2    50   ~ 0
-~WE~
 $EndSCHEMATC
